File: hardware/RevA/marine-tracker-RevA.kicad_pcb (KiCad board)
At the start: 4 copper layers, 73 x 50 mm, 115 parts, among them J1 USB-C, J2 BATTERY, J3 LTE_U.FL, J4 GNSS_L1_L5_U.FL, J5 Nano_SIM, Q1 AO3401A_REVERSE_POLARITY, Q2 MMBT2222A, U1 A7670G-LABE, U10 TPS3808G09DBVR, U11 TPL5111DDCR, U12 SN74LVC2G08DCUR, U13 SN74LVC1G14DBVR, U2 LC29H-AA, U3 BQ24074RGTR, U4 TPS7A2033PDBV, U5 TXS0104EPW, U6 W25Q32JWSSIM, U7 TPS22917DBV_GNSS_LOAD, U8 TPL5010_10MIN_WATCHDOG, U9 TPS3839K33DBZR

Commit message: Route Batch 2 recovery circuit
Routing:
- net PWRKEY: track 0.00 -> 52.8 mm, vias 0 -> 1
- net VSYS: track 0.00 -> 50.1 mm
- net MODEM_RESET_N: track 0.00 -> 42.6 mm
- net WDT_RST_TRIG: track 0.00 -> 42.3 mm
- net GND: track 0.00 -> 36.2 mm, vias 8 -> 10
- net SUPV_TRIG: track 0.00 -> 22.9 mm
- net PWRKEY_TRIG: track 0.00 -> 20.9 mm
- net STRETCH_CT: track 0.00 -> 18.6 mm
- net PWRKEY_ARM_DLY: track 0.00 -> 9.22 mm
- net PWRKEY_ARM: track 0.00 -> 4.71 mm
- net PWRKEY_ARM_DLY_N: track 0.00 -> 4.45 mm
- net AUTO_PWRKEY_BASE: track 0.00 -> 4.01 mm
- net AUTO_PWRKEY_DRV: track 0.00 -> 3.04 mm

Commit message: Repair RevA Batch 2 routing
Routing:
- net GND: track 36.2 -> 26.2 mm, vias 10 -> 14
- net AUTO_PWRKEY_DRV: track 3.04 -> 3.89 mm
- net STRETCH_CT: track 18.6 -> 19.0 mm, vias 0 -> 2
Changed lines of the file:
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@@
 	(segment
 		(start 38.1 36.75)
-		(end 38.5 34.2)
-		(width 0.25)
-		(layer "F.Cu")
-		(net "GND")
-	)
-	(segment
-		(start 40.1375 44.8)
-		(end 43.0625 44.8)
+		(end 38.1 36.95)
+		(width 0.25)
+		(layer "F.Cu")
+		(net "GND")
+	)
+	(segment
+		(start 40.1375 42.9)
+		(end 40.2 42.9)
 		(width 0.25)
 		(layer "F.Cu")
@@
 	)
 	(segment
-		(start 37.8625 43.85)
-		(end 40.1375 44.8)
+		(start 43.0625 44.8)
+		(end 43.2 44.8)
 		(width 0.25)
 		(layer "F.Cu")
@@
 	)
 	(segment
-		(start 37.8625 43.85)
-		(end 40.1375 42.9)
+		(start 40.1375 44.8)
+		(end 40.2 44.8)
 		(width 0.25)
 		(layer "F.Cu")
@@
 	)
 	(via
+		(at 43.2 44.8)
+		(size 0.6)
+		(drill 0.3)
+		(layers "F.Cu" "B.Cu")
+		(net "GND")
+	)
+	(via
+		(at 40.2 42.9)
+		(size 0.6)
+		(drill 0.3)
+		(layers "F.Cu" "B.Cu")
+		(net "GND")
+	)
+	(via
+		(at 38.1 36.95)
+		(size 0.6)
+		(drill 0.3)
+		(layers "F.Cu" "B.Cu")
+		(net "GND")
+	)
+	(via
+		(at 40.2 44.8)
+		(size 0.6)
+		(drill 0.3)
+		(layers "F.Cu" "B.Cu")
+		(net "GND")
+	)
+	(via
 		(at 37.8625 41.77)
 		(size 0.8)
@@
 	(segment
 		(start 40.1375 32.95)
+		(end 41.3 32.6)
+		(width 0.25)
+		(layer "F.Cu")
+		(net "STRETCH_CT")
+	)
+	(segment
+		(start 57.3 27.4)
 		(end 58.05 28)
 		(width 0.25)
 		(layer "F.Cu")
+		(net "STRETCH_CT")
+	)
+	(via
+		(at 41.3 32.6)
+		(size 0.6)
+		(drill 0.3)
+		(layers "F.Cu" "B.Cu")
+		(net "STRETCH_CT")
+	)
+	(via
+		(at 57.3 27.4)
+		(size 0.6)
+		(drill 0.3)
+		(layers "F.Cu" "B.Cu")
+		(net "STRETCH_CT")
+	)
+	(segment
+		(start 41.3 32.6)
+		(end 57.3 27.4)
+		(width 0.25)
+		(layer "B.Cu")
 		(net "STRETCH_CT")
 	)
@@
 	(segment
 		(start 40.1375 43.85)
+		(end 41.5 44.4)
+		(width 0.25)
+		(layer "F.Cu")
+		(net "AUTO_PWRKEY_DRV")
+	)
+	(segment
+		(start 41.5 44.4)
 		(end 40.99 46.77)
 		(width 0.25)

Commit message: Fix RevA Batch A routing defects
Routing:
- net VSYS: track 50.1 -> 58.0 mm, vias 0 -> 2
- net PWRKEY_ARM_DLY: track 9.22 -> 11.0 mm, vias 0 -> 2
Changed lines of the file:
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@@
 	(segment
 		(start 43.51 32)
-		(end 43.02 36)
-		(width 0.4)
+		(end 43.51 31.3)
+		(width 0.25)
 		(layer "F.Cu")
 		(net "VSYS")
@@
 	)
 	(segment
+		(start 43.02 34)
+		(end 43.02 36)
+		(width 0.25)
+		(layer "F.Cu")
+		(net "VSYS")
+	)
+	(segment
 		(start 43.02 36)
 		(end 40.9 35.25)
 		(width 0.4)
 		(layer "F.Cu")
+		(net "VSYS")
+	)
+	(via
+		(at 43.02 34)
+		(size 0.6)
+		(drill 0.3)
+		(layers "F.Cu" "B.Cu")
+		(net "VSYS")
+	)
+	(via
+		(at 43.51 31.3)
+		(size 0.6)
+		(drill 0.3)
+		(layers "F.Cu" "B.Cu")
+		(net "VSYS")
+	)
+	(segment
+		(start 40 31.3)
+		(end 40 34)
+		(width 0.25)
+		(layer "B.Cu")
+		(net "VSYS")
+	)
+	(segment
+		(start 40 34)
+		(end 43.02 34)
+		(width 0.25)
+		(layer "B.Cu")
+		(net "VSYS")
+	)
+	(segment
+		(start 43.51 31.3)
+		(end 40 31.3)
+		(width 0.25)
+		(layer "B.Cu")
 		(net "VSYS")
 	)
@@
 	)
 	(segment
+		(start 37.3 39.7)
+		(end 37.9625 39.7)
+		(width 0.25)
+		(layer "F.Cu")
+		(net "PWRKEY_ARM_DLY")
+	)
+	(segment
 		(start 44.51 38.4)
-		(end 37.9625 39.7)
+		(end 44.51 38.9)
 		(width 0.25)
 		(layer "F.Cu")
@@
 		(net "PWRKEY_ARM_DLY")
 	)
+	(via
+		(at 37.3 39.7)
+		(size 0.6)
+		(drill 0.3)
+		(layers "F.Cu" "B.Cu")
+		(net "PWRKEY_ARM_DLY")
+	)
+	(via
+		(at 44.51 38.9)
+		(size 0.6)
+		(drill 0.3)
+		(layers "F.Cu" "B.Cu")
+		(net "PWRKEY_ARM_DLY")
+	)
+	(segment
+		(start 44.51 38.9)
+		(end 37.3 39.7)
+		(width 0.25)
+		(layer "B.Cu")
+		(net "PWRKEY_ARM_DLY")
+	)
